File: hardware/v2/tappytap.brd (EAGLE design)
At the start: 36 x 16 mm, 18 parts

Commit message: Fix spacing issue for pcbway
Parts:
- HBR1, HBR2, HBR3: device Sparky:24-SSOP -> Sparky:SSOP-24
Routing:
- net GND: track 156.8 -> 156.1 mm
