File: hardware/v3/tappytap.sch (EAGLE design)
At the start: 18 parts

Commit message: Tappytap v3 design done with gerbers
Parts:
- removed DATA_IN, DATA_OUT: (no value), SparkFun-Connectors:CONN_05
- added IN, OUT: (no value), SparkFun-Connectors:CONN_06SILK_FEMALE_PTH
Connections:
- new net V+: HBR1.VS1, HBR1.VS2, HBR2.VS1, HBR2.VS2, HBR3.VS1, HBR3.VS2, IN.6, OUT.6
- net +5V: now also IN.5, OUT.5; no longer DATA_IN.5, DATA_OUT.5, HBR1.VS1, HBR1.VS2, HBR2.VS1, HBR2.VS2, HBR3.VS1, HBR3.VS2
- net GND: now also IN.1, OUT.1; no longer DATA_IN.1, DATA_OUT.1
- net NCV_CS: now also IN.2, OUT.2; no longer DATA_IN.2, DATA_OUT.2
- net SCK: now also IN.3, OUT.3; no longer DATA_IN.3, DATA_OUT.3
- net SI: now also IN.4; no longer DATA_IN.4
- net SO: now also OUT.4; no longer DATA_OUT.4
