File: hardware/v4-sur/tappytap.brd (EAGLE design)
At the start: 36 x 37 mm, 18 parts

Commit message: Ship v4-sur
Parts:
- flipped IN to the bottom
- flipped OUT to the bottom
Routing:
- net V+: track 98.4 -> 94.3 mm, vias 6 -> 5
- net GND: track 152.4 -> 149.1 mm, vias 7 -> 5
- net SCK: track 60.3 -> 62.0 mm, vias 3 -> 4
- net SI: track 10.9 -> 11.3 mm, vias 1 -> 2
- net NCV_CS: track 58.4 -> 58.5 mm, vias 3 -> 4
- net +5V: track 86.8 -> 86.9 mm, vias 2 -> 4
- net SO: vias 1 -> 0
