File: hardware/v6-flex/tappytap_v6_AoA_6x6.brd (EAGLE design)
At the start: 45.8 x 46 mm, 60 parts, among them X1 52746-6, X2 52746-6, X3 52746-6, X4 52746-6

Commit message: Gerbers and some related tweaks
Other:
- board size 45.8 x 46 mm -> 46 x 46 mm
