File: hardware/v7-flex2811/v7-flex2811_long.sch (EAGLE design)
At the start: 128 parts

Commit message: first draft tapper strip
Parts:
- removed U$3: 4PAD, Sparky:4PAD
- added C17, C18, C19, C20: (no value), rcl:C-EUC0201
- added IN1, U$67, U$68, U$71, U$72, U$75, U$76, U$79, U$80: 4PAD, Sparky:4PAD
- added R49, R50, R51, R52, R53, R54, R55, R56, R57, R58, R59, R60: (no value), rcl:R-US_R0201
- added U$65, U$69, U$73, U$77: TP_4MM_MED_PAD, tom-tappytap-v5-flex:TP_4MM_MED_PAD
- added U$66, U$70, U$74, U$78: WS2818, adafruit:WS2818
- renumbered U$4 to OUT1
Connections:
- removed net BIN: U$10.BIN, U$11.P$2, U$14.BIN, U$15.P$2, U$18.BIN, U$19.P$2, U$2.BIN, U$22.BIN, U$23.P$2, U$26.BIN, U$27.P$2, U$3.P$2, U$30.BIN, U$31.P$2, U$34.BIN, U$35.P$2, U$38.BIN, U$39.P$2, U$42.BIN, U$43.P$2, U$46.BIN, U$47.P$2, U$50.BIN, U$51.P$2, U$54.BIN, U$55.P$2, U$58.BIN, U$59.P$2, U$6.BIN, U$62.BIN, U$63.P$2, U$7.P$2
- removed net DIN: OUT1.P$2, R1.2, R10.2, R13.2, R16.2, R19.2, R22.2, R25.2, R28.2, R31.2, R34.2, R37.2, R4.2, R40.2, R43.2, R46.2, R7.2, U$11.P$1, U$12.P$2, U$15.P$1, U$16.P$2, U$19.P$1, U$20.P$2, U$23.P$1, U$24.P$2, U$27.P$1, U$28.P$2, U$3.P$1, U$31.P$1, U$32.P$2, U$35.P$1, U$36.P$2, U$39.P$1, U$40.P$2, U$43.P$1, U$44.P$2, U$47.P$1, U$48.P$2, U$51.P$1, U$52.P$2, U$55.P$1, U$56.P$2, U$59.P$1, U$60.P$2, U$63.P$1, U$64.P$2, U$7.P$1, U$8.P$2
- removed net DOUT: OUT1.P$1, R11.1, R14.1, R17.1, R2.1, R20.1, R23.1, R26.1, R29.1, R32.1, R35.1, R38.1, R41.1, R44.1, R47.1, R5.1, R8.1, U$12.P$1, U$16.P$1, U$20.P$1, U$24.P$1, U$28.P$1, U$32.P$1, U$36.P$1, U$40.P$1, U$44.P$1, U$48.P$1, U$52.P$1, U$56.P$1, U$60.P$1, U$64.P$1, U$8.P$1
- removed net NEG_PAD: U$1.0, U$10.OUTB, U$10.OUTG, U$10.OUTR, U$13.0, U$14.OUTB, U$14.OUTG, U$14.OUTR, U$17.0, U$18.OUTB, U$18.OUTG, U$18.OUTR, U$2.OUTB, U$2.OUTG, U$2.OUTR, U$21.0, U$22.OUTB, U$22.OUTG, U$22.OUTR, U$25.0, U$26.OUTB, U$26.OUTG, U$26.OUTR, U$29.0, U$30.OUTB, U$30.OUTG, U$30.OUTR, U$33.0, U$34.OUTB, U$34.OUTG, U$34.OUTR, U$37.0, U$38.OUTB, U$38.OUTG, U$38.OUTR, U$41.0, U$42.OUTB, U$42.OUTG, U$42.OUTR, U$45.0, U$46.OUTB, U$46.OUTG, U$46.OUTR, U$49.0, U$5.0, U$50.OUTB, U$50.OUTG, U$50.OUTR, U$53.0, U$54.OUTB, U$54.OUTG, U$54.OUTR, U$57.0, U$58.OUTB, U$58.OUTG, U$58.OUTR, U$6.OUTB, U$6.OUTG, U$6.OUTR, U$61.0, U$62.OUTB, U$62.OUTG, U$62.OUTR, U$9.0
- new net BIN1: IN1.BIN, U$2.BIN
- new net DIN1: IN1.DIN, OUT1.BIN, R4.2, U$6.BIN, U$7.BIN
- new net DOUT1: OUT1.DIN, R1.2, R5.1, U$10.BIN, U$11.BIN, U$7.DIN, U$8.BIN
- new net DOUT10: R29.1, R31.2, U$40.DIN, U$43.DIN, U$44.BIN, U$46.BIN, U$47.BIN
- new net DOUT11: R32.1, R34.2, U$44.DIN, U$47.DIN, U$48.BIN, U$50.BIN, U$51.BIN
- new net DOUT12: R35.1, R37.2, U$48.DIN, U$51.DIN, U$52.BIN, U$54.BIN, U$55.BIN
- new net DOUT13: R38.1, R40.2, U$52.DIN, U$55.DIN, U$56.BIN, U$58.BIN, U$59.BIN
- new net DOUT14: R41.1, R43.2, U$56.DIN, U$59.DIN, U$60.BIN, U$62.BIN, U$63.BIN
- new net DOUT15: R44.1, R46.2, U$60.DIN, U$63.DIN, U$64.BIN, U$66.BIN, U$67.BIN
- new net DOUT16: R47.1, R49.2, U$64.DIN, U$67.DIN, U$68.BIN, U$70.BIN, U$71.BIN
- new net DOUT17: R50.1, R52.2, U$68.DIN, U$71.DIN, U$72.BIN, U$74.BIN, U$75.BIN
- new net DOUT18: R53.1, R55.2, U$72.DIN, U$75.DIN, U$76.BIN, U$78.BIN, U$79.BIN
- new net DOUT19: R56.1, R58.2, U$76.DIN, U$79.DIN, U$80.BIN
- new net DOUT2: R2.1, R7.2, U$11.DIN, U$12.BIN, U$14.BIN, U$15.BIN, U$8.DIN
- new net DOUT20: R59.1, U$80.DIN
- new net DOUT3: R10.2, R8.1, U$12.DIN, U$15.DIN, U$16.BIN, U$18.BIN, U$19.BIN
- new net DOUT4: R11.1, R13.2, U$16.DIN, U$19.DIN, U$20.BIN, U$22.BIN, U$23.BIN
- new net DOUT5: R14.1, R16.2, U$20.DIN, U$23.DIN, U$24.BIN, U$26.BIN, U$27.BIN
- new net DOUT6: R17.1, R19.2, U$24.DIN, U$27.DIN, U$28.BIN, U$30.BIN, U$31.BIN
- new net DOUT7: R20.1, R22.2, U$28.DIN, U$31.DIN, U$32.BIN, U$34.BIN, U$35.BIN
- new net DOUT8: R23.1, R25.2, U$32.DIN, U$35.DIN, U$36.BIN, U$38.BIN, U$39.BIN
- new net DOUT9: R26.1, R28.2, U$36.DIN, U$39.DIN, U$40.BIN, U$42.BIN, U$43.BIN
- new net N$49: R49.1, U$66.DIN
- new net N$50: R50.2, U$66.DO
- new net N$51: R51.1, U$66.VDD
- new net N$52: R52.1, U$70.DIN
- new net N$53: R53.2, U$70.DO
- new net N$54: R54.1, U$70.VDD
- new net N$55: R55.1, U$74.DIN
- new net N$56: R56.2, U$74.DO
- new net N$57: R57.1, U$74.VDD
- new net N$58: R58.1, U$78.DIN
- new net N$59: R59.2, U$78.DO
- new net N$60: R60.1, U$78.VDD
- new net NEG_PAD1: U$1.0, U$2.OUTB, U$2.OUTG, U$2.OUTR
- new net NEG_PAD10: U$37.0, U$38.OUTB, U$38.OUTG, U$38.OUTR
- new net NEG_PAD11: U$41.0, U$42.OUTB, U$42.OUTG, U$42.OUTR
- new net NEG_PAD12: U$45.0, U$46.OUTB, U$46.OUTG, U$46.OUTR
- new net NEG_PAD13: U$49.0, U$50.OUTB, U$50.OUTG, U$50.OUTR
- new net NEG_PAD14: U$53.0, U$54.OUTB, U$54.OUTG, U$54.OUTR
- new net NEG_PAD15: U$57.0, U$58.OUTB, U$58.OUTG, U$58.OUTR
- new net NEG_PAD16: U$61.0, U$62.OUTB, U$62.OUTG, U$62.OUTR
- new net NEG_PAD17: U$65.0, U$66.OUTB, U$66.OUTG, U$66.OUTR
- new net NEG_PAD18: U$69.0, U$70.OUTB, U$70.OUTG, U$70.OUTR
- new net NEG_PAD19: U$73.0, U$74.OUTB, U$74.OUTG, U$74.OUTR
- new net NEG_PAD2: U$5.0, U$6.OUTB, U$6.OUTG, U$6.OUTR
- new net NEG_PAD20: U$77.0, U$78.OUTB, U$78.OUTG, U$78.OUTR
- new net NEG_PAD3: U$10.OUTB, U$10.OUTG, U$10.OUTR, U$9.0
- new net NEG_PAD4: U$13.0, U$14.OUTB, U$14.OUTG, U$14.OUTR
- new net NEG_PAD5: U$17.0, U$18.OUTB, U$18.OUTG, U$18.OUTR
- new net NEG_PAD6: U$21.0, U$22.OUTB, U$22.OUTG, U$22.OUTR
- new net NEG_PAD7: U$25.0, U$26.OUTB, U$26.OUTG, U$26.OUTR
- new net NEG_PAD8: U$29.0, U$30.OUTB, U$30.OUTG, U$30.OUTR
- new net NEG_PAD9: U$33.0, U$34.OUTB, U$34.OUTG, U$34.OUTR
- net GND: now also C17.2, C18.2, C19.2, C20.2, IN1.GND, OUT1.GND, U$11.GND, U$12.GND, U$15.GND, U$16.GND, U$19.GND, U$20.GND, U$23.GND, U$24.GND, U$27.GND, U$28.GND, U$31.GND, U$32.GND, U$35.GND, U$36.GND, U$39.GND, U$40.GND, U$43.GND, U$44.GND, U$47.GND, U$48.GND, U$51.GND, U$52.GND, U$55.GND, U$56.GND, U$59.GND, U$60.GND, U$63.GND, U$64.GND, U$66.GND, U$67.GND, U$68.GND, U$7.GND, U$70.GND, U$71.GND, U$72.GND, U$74.GND, U$75.GND, U$76.GND, U$78.GND, U$79.GND, U$8.GND, U$80.GND; no longer OUT1.P$3, U$11.P$3, U$12.P$3, U$15.P$3, U$16.P$3, U$19.P$3, U$20.P$3, U$23.P$3, U$24.P$3, U$27.P$3, U$28.P$3, U$3.P$3, U$31.P$3, U$32.P$3, U$35.P$3, U$36.P$3, U$39.P$3, U$40.P$3, U$43.P$3, U$44.P$3, U$47.P$3, U$48.P$3, U$51.P$3, U$52.P$3, U$55.P$3, U$56.P$3, U$59.P$3, U$60.P$3, U$63.P$3, U$64.P$3, U$7.P$3, U$8.P$3
- net VCC: now also C17.1, C18.1, C19.1, C20.1, IN1.VCC, OUT1.VCC, R51.2, R54.2, R57.2, R60.2, U$11.VCC, U$12.VCC, U$15.VCC, U$16.VCC, U$19.VCC, U$20.VCC, U$23.VCC, U$24.VCC, U$27.VCC, U$28.VCC, U$31.VCC, U$32.VCC, U$35.VCC, U$36.VCC, U$39.VCC, U$40.VCC, U$43.VCC, U$44.VCC, U$47.VCC, U$48.VCC, U$51.VCC, U$52.VCC, U$55.VCC, U$56.VCC, U$59.VCC, U$60.VCC, U$63.VCC, U$64.VCC, U$65.1, U$67.VCC, U$68.VCC, U$69.1, U$7.VCC, U$71.VCC, U$72.VCC, U$73.1, U$75.VCC, U$76.VCC, U$77.1, U$79.VCC, U$8.VCC, U$80.VCC; no longer OUT1.P$4, U$11.P$4, U$12.P$4, U$15.P$4, U$16.P$4, U$19.P$4, U$20.P$4, U$23.P$4, U$24.P$4, U$27.P$4, U$28.P$4, U$3.P$4, U$31.P$4, U$32.P$4, U$35.P$4, U$36.P$4, U$39.P$4, U$40.P$4, U$43.P$4, U$44.P$4, U$47.P$4, U$48.P$4, U$51.P$4, U$52.P$4, U$55.P$4, U$56.P$4, U$59.P$4, U$60.P$4, U$63.P$4, U$64.P$4, U$7.P$4, U$8.P$4
