File: hardware/v7-flex2811/v7-flex2811_32x.brd (EAGLE design)
At the start: 248 x 7.8 mm, 256 parts

Commit message: More edit for manufacturability
Add a preliminary BOM
Add labels for the ICs for assembly
Parts:
- R12, R15, R18, R21, R24, R27, R3, R30, R33, R36, R39, R42, R45, R48, R51, R54, R57, R6, R60, R63, R66, R69, R72, R75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: value (none) -> 100
- renumbered U$10 to U3, U$102 to U26, U$106 to U27, U$110 to U28, U$114 to U29, U$118 to U30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
