File: hardware/v7-flex2811/v7-flex2811_single.sch (EAGLE design)
At the start: 128 parts

Commit message: first draft tapper strip
Parts:
- removed C1, C10, C11, C12, C13, C14, C15, C16, C3, C4, C5, C6, C7, C8, C9: (no value), rcl:C-EUC0201
- removed R1, R10, R11, R12, R13, R14, R15, R16, R17, R18, R19, R2, R20, R21, R22, R23, R24, R25, R26, R27, R28, R29, R3, R30, R31, R32, R33, R34, R35, R36, R37, R38, R39, R40, R41, R42, R43, R44, R45, R46, R47, R48, R7, R8, R9: (no value), rcl:R-US_R0201
- removed U$10, U$14, U$18, U$22, U$26, U$30, U$34, U$38, U$42, U$46, U$50, U$54, U$58, U$6, U$62: WS2818, adafruit:WS2818
- removed U$11, U$12, U$15, U$16, U$19, U$20, U$23, U$24, U$27, U$28, U$31, U$32, U$35, U$36, U$39, U$40, U$43, U$44, U$47, U$48, U$51, U$52, U$55, U$56, U$59, U$60, U$63, U$64, U$7, U$8: 4PAD, Sparky:4PAD
- removed U$13, U$17, U$21, U$25, U$29, U$33, U$37, U$41, U$45, U$49, U$5, U$53, U$57, U$61, U$9: TP_4MM_MED_PAD, tom-tappytap-v5-flex:TP_4MM_MED_PAD
Connections:
- removed net N$1: R1.1, U$6.DIN
- removed net N$10: R10.1, U$14.DIN
- removed net N$11: R11.2, U$14.DO
- removed net N$12: R12.1, U$14.VDD
- removed net N$13: R13.1, U$18.DIN
- removed net N$14: R14.2, U$18.DO
- removed net N$15: R15.1, U$18.VDD
- removed net N$16: R16.1, U$22.DIN
- removed net N$17: R17.2, U$22.DO
- removed net N$18: R18.1, U$22.VDD
- removed net N$19: R19.1, U$26.DIN
- removed net N$2: R2.2, U$6.DO
- removed net N$20: R20.2, U$26.DO
- removed net N$21: R21.1, U$26.VDD
- removed net N$22: R22.1, U$30.DIN
- removed net N$23: R23.2, U$30.DO
- removed net N$24: R24.1, U$30.VDD
- removed net N$25: R25.1, U$34.DIN
- removed net N$26: R26.2, U$34.DO
- removed net N$27: R27.1, U$34.VDD
- removed net N$28: R28.1, U$38.DIN
- removed net N$29: R29.2, U$38.DO
- removed net N$3: R3.1, U$6.VDD
- removed net N$30: R30.1, U$38.VDD
- removed net N$31: R31.1, U$42.DIN
- removed net N$32: R32.2, U$42.DO
- removed net N$33: R33.1, U$42.VDD
- removed net N$34: R34.1, U$46.DIN
- removed net N$35: R35.2, U$46.DO
- removed net N$36: R36.1, U$46.VDD
- removed net N$37: R37.1, U$50.DIN
- removed net N$38: R38.2, U$50.DO
- removed net N$39: R39.1, U$50.VDD
- removed net N$40: R40.1, U$54.DIN
- removed net N$41: R41.2, U$54.DO
- removed net N$42: R42.1, U$54.VDD
- removed net N$43: R43.1, U$58.DIN
- removed net N$44: R44.2, U$58.DO
- removed net N$45: R45.1, U$58.VDD
- removed net N$46: R46.1, U$62.DIN
- removed net N$47: R47.2, U$62.DO
- removed net N$48: R48.1, U$62.VDD
- removed net N$7: R7.1, U$10.DIN
- removed net N$8: R8.2, U$10.DO
- removed net N$9: R9.1, U$10.VDD
- net BIN: no longer U$10.BIN, U$11.P$2, U$14.BIN, U$15.P$2, U$18.BIN, U$19.P$2, U$22.BIN, U$23.P$2, U$26.BIN, U$27.P$2, U$30.BIN, U$31.P$2, U$34.BIN, U$35.P$2, U$38.BIN, U$39.P$2, U$42.BIN, U$43.P$2, U$46.BIN, U$47.P$2, U$50.BIN, U$51.P$2, U$54.BIN, U$55.P$2, U$58.BIN, U$59.P$2, U$6.BIN, U$62.BIN, U$63.P$2, U$7.P$2
- net DIN: no longer R1.2, R10.2, R13.2, R16.2, R19.2, R22.2, R25.2, R28.2, R31.2, R34.2, R37.2, R40.2, R43.2, R46.2, R7.2, U$11.P$1, U$12.P$2, U$15.P$1, U$16.P$2, U$19.P$1, U$20.P$2, U$23.P$1, U$24.P$2, U$27.P$1, U$28.P$2, U$31.P$1, U$32.P$2, U$35.P$1, U$36.P$2, U$39.P$1, U$40.P$2, U$43.P$1, U$44.P$2, U$47.P$1, U$48.P$2, U$51.P$1, U$52.P$2, U$55.P$1, U$56.P$2, U$59.P$1, U$60.P$2, U$63.P$1, U$64.P$2, U$7.P$1, U$8.P$2
- net DOUT: no longer R11.1, R14.1, R17.1, R2.1, R20.1, R23.1, R26.1, R29.1, R32.1, R35.1, R38.1, R41.1, R44.1, R47.1, R8.1, U$12.P$1, U$16.P$1, U$20.P$1, U$24.P$1, U$28.P$1, U$32.P$1, U$36.P$1, U$40.P$1, U$44.P$1, U$48.P$1, U$52.P$1, U$56.P$1, U$60.P$1, U$64.P$1, U$8.P$1
- net GND: no longer C1.2, C10.2, C11.2, C12.2, C13.2, C14.2, C15.2, C16.2, C3.2, C4.2, C5.2, C6.2, C7.2, C8.2, C9.2, U$10.GND, U$11.P$3, U$12.P$3, U$14.GND, U$15.P$3, U$16.P$3, U$18.GND, U$19.P$3, U$20.P$3, U$22.GND, U$23.P$3, U$24.P$3, U$26.GND, U$27.P$3, U$28.P$3, U$30.GND, U$31.P$3, U$32.P$3, U$34.GND, U$35.P$3, U$36.P$3, U$38.GND, U$39.P$3, U$40.P$3, U$42.GND, U$43.P$3, U$44.P$3, U$46.GND, U$47.P$3, U$48.P$3, U$50.GND, U$51.P$3, U$52.P$3, U$54.GND, U$55.P$3, U$56.P$3, U$58.GND, U$59.P$3, U$6.GND, U$60.P$3, U$62.GND, U$63.P$3, U$64.P$3, U$7.P$3, U$8.P$3
- net NEG_PAD: no longer U$10.OUTB, U$10.OUTG, U$10.OUTR, U$13.0, U$14.OUTB, U$14.OUTG, U$14.OUTR, U$17.0, U$18.OUTB, U$18.OUTG, U$18.OUTR, U$21.0, U$22.OUTB, U$22.OUTG, U$22.OUTR, U$25.0, U$26.OUTB, U$26.OUTG, U$26.OUTR, U$29.0, U$30.OUTB, U$30.OUTG, U$30.OUTR, U$33.0, U$34.OUTB, U$34.OUTG, U$34.OUTR, U$37.0, U$38.OUTB, U$38.OUTG, U$38.OUTR, U$41.0, U$42.OUTB, U$42.OUTG, U$42.OUTR, U$45.0, U$46.OUTB, U$46.OUTG, U$46.OUTR, U$49.0, U$5.0, U$50.OUTB, U$50.OUTG, U$50.OUTR, U$53.0, U$54.OUTB, U$54.OUTG, U$54.OUTR, U$57.0, U$58.OUTB, U$58.OUTG, U$58.OUTR, U$6.OUTB, U$6.OUTG, U$6.OUTR, U$61.0, U$62.OUTB, U$62.OUTG, U$62.OUTR, U$9.0
- net VCC: no longer C1.1, C10.1, C11.1, C12.1, C13.1, C14.1, C15.1, C16.1, C3.1, C4.1, C5.1, C6.1, C7.1, C8.1, C9.1, R12.2, R15.2, R18.2, R21.2, R24.2, R27.2, R3.2, R30.2, R33.2, R36.2, R39.2, R42.2, R45.2, R48.2, R9.2, U$11.P$4, U$12.P$4, U$13.1, U$15.P$4, U$16.P$4, U$17.1, U$19.P$4, U$20.P$4, U$21.1, U$23.P$4, U$24.P$4, U$25.1, U$27.P$4, U$28.P$4, U$29.1, U$31.P$4, U$32.P$4, U$33.1, U$35.P$4, U$36.P$4, U$37.1, U$39.P$4, U$40.P$4, U$41.1, U$43.P$4, U$44.P$4, U$45.1, U$47.P$4, U$48.P$4, U$49.1, U$5.1, U$51.P$4, U$52.P$4, U$53.1, U$55.P$4, U$56.P$4, U$57.1, U$59.P$4, U$60.P$4, U$61.1, U$63.P$4, U$64.P$4, U$7.P$4, U$8.P$4, U$9.1

Commit message: Rework the single for more clearance to make fab easier
Was concerned about how tight the passives were for
assmebly, have just spread it out a bit

Also made the WS2818 pads slightly smaller so we have more clearance
Parts:
- U$2: device adafruit:WS2818 -> Sparky:WS2818
Changed lines of the file:
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@@
 <?xml version="1.0" encoding="utf-8"?>
 <!DOCTYPE eagle SYSTEM "eagle.dtd">
-<eagle version="6.5.0">
+<eagle version="7.3.0">
 <drawing>
 <settings>
@@
 <grid distance="0.1" unitdist="inch" unit="inch" style="lines" multiple="1" display="no" altdistance="0.01" altunitdist="inch" altunit="inch"/>
 <layers>
-<layer number="1" name="Top" color="4" fill="1" visible="yes" active="no"/>
-<layer number="2" name="Route2" color="1" fill="3" visible="yes" active="no"/>
-<layer number="3" name="Route3" color="4" fill="3" visible="yes" active="no"/>
-<layer number="4" name="Route4" color="1" fill="4" visible="yes" active="no"/>
-<layer number="5" name="Route5" color="4" fill="4" visible="yes" active="no"/>
-<layer number="6" name="Route6" color="1" fill="8" visible="yes" active="no"/>
-<layer number="7" name="Route7" color="4" fill="8" visible="yes" active="no"/>
-<layer number="8" name="Route8" color="1" fill="2" visible="yes" active="no"/>
-<layer number="9" name="Route9" color="4" fill="2" visible="yes" active="no"/>
-<layer number="10" name="Route10" color="1" fill="7" visible="yes" active="no"/>
-<layer number="11" name="Route11" color="4" fill="7" visible="yes" active="no"/>
-<layer number="12" name="Route12" color="1" fill="5" visible="yes" active="no"/>
-<layer number="13" name="Route13" color="4" fill="5" visible="yes" active="no"/>
-<layer number="14" name="Route14" color="1" fill="6" visible="yes" active="no"/>
-<layer number="15" name="Route15" color="4" fill="6" visible="yes" active="no"/>
-<layer number="16" name="Bottom" color="1" fill="1" visible="yes" active="no"/>
-<layer number="17" name="Pads" color="2" fill="1" visible="yes" active="no"/>
-<layer number="18" name="Vias" color="2" fill="1" visible="yes" active="no"/>
-<layer number="19" name="Unrouted" color="6" fill="1" visible="yes" active="no"/>
-<layer number="20" name="Dimension" color="15" fill="1" visible="yes" active="no"/>
-<layer number="21" name="tPlace" color="7" fill="1" visible="yes" active="no"/>
-<layer number="22" name="bPlace" color="7" fill="1" visible="yes" active="no"/>
-<layer number="23" name="tOrigins" color="15" fill="1" visible="yes" active="no"/>
-<layer number="24" name="bOrigins" color="15" fill="1" visible="yes" active="no"/>
-<layer number="25" name="tNames" color="7" fill="1" visible="yes" active="no"/>
-<layer number="26" name="bNames" color="7" fill="1" visible="yes" active="no"/>
-<layer number="27" name="tValues" color="7" fill="1" visible="yes" active="no"/>
-<layer number="28" name="bValues" color="7" fill="1" visible="yes" active="no"/>
+<layer number="1" name="Top" color="4" fill="1" visible="no" active="no"/>
+<layer number="2" name="Route2" color="1" fill="3" visible="no" active="no"/>
+<layer number="3" name="Route3" color="4" fill="3" visible="no" active="no"/>
+<layer number="4" name="Route4" color="1" fill="4" visible="no" active="no"/>
+<layer number="5" name="Route5" color="4" fill="4" visible="no" active="no"/>
+<layer number="6" name="Route6" color="1" fill="8" visible="no" active="no"/>
+<layer number="7" name="Route7" color="4" fill="8" visible="no" active="no"/>
+<layer number="8" name="Route8" color="1" fill="2" visible="no" active="no"/>
+<layer number="9" name="Route9" color="4" fill="2" visible="no" active="no"/>
+<layer number="10" name="Route10" color="1" fill="7" visible="no" active="no"/>
+<layer number="11" name="Route11" color="4" fill="7" visible="no" active="no"/>
+<layer number="12" name="Route12" color="1" fill="5" visible="no" active="no"/>
+<layer number="13" name="Route13" color="4" fill="5" visible="no" active="no"/>
+<layer number="14" name="Route14" color="1" fill="6" visible="no" active="no"/>
+<layer number="15" name="Route15" color="4" fill="6" visible="no" active="no"/>
+<layer number="16" name="Bottom" color="1" fill="1" visible="no" active="no"/>
+<layer number="17" name="Pads" color="2" fill="1" visible="no" active="no"/>
+<layer number="18" name="Vias" color="2" fill="1" visible="no" active="no"/>
+<layer number="19" name="Unrouted" color="6" fill="1" visible="no" active="no"/>
+<layer number="20" name="Dimension" color="15" fill="1" visible="no" active="no"/>
+<layer number="21" name="tPlace" color="7" fill="1" visible="no" active="no"/>
+<layer number="22" name="bPlace" color="7" fill="1" visible="no" active="no"/>
+<layer number="23" name="tOrigins" color="15" fill="1" visible="no" active="no"/>
+<layer number="24" name="bOrigins" color="15" fill="1" visible="no" active="no"/>
+<layer number="25" name="tNames" color="7" fill="1" visible="no" active="no"/>
+<layer number="26" name="bNames" color="7" fill="1" visible="no" active="no"/>
+<layer number="27" name="tValues" color="7" fill="1" visible="no" active="no"/>
+<layer number="28" name="bValues" color="7" fill="1" visible="no" active="no"/>
 <layer number="29" name="tStop" color="7" fill="3" visible="no" active="no"/>
 <layer number="30" name="bStop" color="7" fill="6" visible="no" active="no"/>
@@
 <layer number="35" name="tGlue" color="7" fill="4" visible="no" active="no"/>
 <layer number="36" name="bGlue" color="7" fill="5" visible="no" active="no"/>
-<layer number="37" name="tTest" color="7" fill="1" visible="yes" active="no"/>
-<layer number="38" name="bTest" color="7" fill="1" visible="yes" active="no"/>
+<layer number="37" name="tTest" color="7" fill="1" visible="no" active="no"/>
+<layer number="38" name="bTest" color="7" fill="1" visible="no" active="no"/>
 <layer number="39" name="tKeepout" color="4" fill="11" visible="no" active="no"/>
 <layer number="40" name="bKeepout" color="1" fill="11" visible="no" active="no"/>
@@
 <layer number="44" name="Drills" color="7" fill="1" visible="no" active="no"/>
 <layer number="45" name="Holes" color="7" fill="1" visible="no" active="no"/>
-<layer number="46" name="Milling" color="3" fill="1" visible="yes" active="no"/>
-<layer number="47" name="Measures" color="7" fill="1" visible="yes" active="no"/>
-<layer number="48" name="Document" color="7" fill="1" visible="yes" active="no"/>
-<layer number="49" name="Reference" color="7" fill="1" visible="yes" active="no"/>
-<layer number="50" name="dxf" color="7" fill="1" visible="yes" active="no"/>
-<layer number="51" name="tDocu" color="7" fill="1" visible="yes" active="no"/>
-<layer number="52" name="bDocu" color="7" fill="1" visible="yes" active="no"/>
-<layer number="53" name="tGND_GNDA" color="7" fill="9" visible="yes" active="no"/>
-<layer number="54" name="bGND_GNDA" color="1" fill="9" visible="yes" active="no"/>
-<layer number="56" name="wert" color="7" fill="1" visible="yes" active="no"/>
-<layer number="57" name="tCAD" color="7" fill="1" visible="yes" active="no"/>
-<layer number="59" name="tCarbon" color="7" fill="1" visible="yes" active="no"/>
-<layer number="60" name="bCarbon" color="7" fill="1" visible="yes" active="no"/>
+<layer number="46" name="Milling" color="3" fill="1" visible="no" active="no"/>
+<layer number="47" name="Measures" color="7" fill="1" visible="no" active="no"/>
+<layer number="48" name="Document" color="7" fill="1" visible="no" active="no"/>
+<layer number="49" name="Reference" color="7" fill="1" visible="no" active="no"/>
+<layer number="50" name="dxf" color="7" fill="1" visible="no" active="no"/>
+<layer number="51" name="tDocu" color="7" fill="1" visible="no" active="no"/>
+<layer number="52" name="bDocu" color="7" fill="1" visible="no" active="no"/>
+<layer number="53" name="tGND_GNDA" color="7" fill="9" visible="no" active="no"/>
+<layer number="54" name="bGND_GNDA" color="1" fill="9" visible="no" active="no"/>
+<layer number="56" name="wert" color="7" fill="1" visible="no" active="no"/>
+<layer number="57" name="tCAD" color="7" fill="1" visible="no" active="no"/>
+<layer number="59" name="tCarbon" color="7" fill="1" visible="no" active="no"/>
+<layer number="60" name="bCarbon" color="7" fill="1" visible="no" active="no"/>
 <layer number="90" name="Modules" color="5" fill="1" visible="yes" active="yes"/>
 <layer number="91" name="Nets" color="2" fill="1" visible="yes" active="yes"/>
@@
 <part name="P+3" library="supply1" deviceset="VCC" device=""/>
 <part name="GND1" library="supply1" deviceset="GND" device=""/>
-<part name="U$2" library="adafruit" deviceset="WS2818" device=""/>
+<part name="U$2" library="Sparky" deviceset="WS2818" device=""/>
 <part name="GND3" library="supply1" deviceset="GND" device=""/>
 <part name="R4" library="rcl" deviceset="R-US_" device="R0201"/>

Commit message: More edit for manufacturability
Add a preliminary BOM
Add labels for the ICs for assembly
Parts:
- C2: value (none) -> 0.1uF
- R4, R5: value (none) -> 33Ω
- R6: value (none) -> 100Ω
- renumbered U$1 to P1, U$2 to U1
Changed lines of the file:
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@@
 </classes>
 <parts>
-<part name="C2" library="rcl" deviceset="C-EU" device="C0201"/>
+<part name="C2" library="rcl" deviceset="C-EU" device="C0201" value="0.1uF"/>
 <part name="P+1" library="supply1" deviceset="VCC" device=""/>
-<part name="U$1" library="tom-tappytap-v5-flex" deviceset="TP_4MM_MED_PAD" device=""/>
+<part name="P1" library="tom-tappytap-v5-flex" deviceset="TP_4MM_MED_PAD" device=""/>
 <part name="P+3" library="supply1" deviceset="VCC" device=""/>
 <part name="GND1" library="supply1" deviceset="GND" device=""/>
-<part name="U$2" library="Sparky" deviceset="WS2818" device=""/>
+<part name="U1" library="Sparky" deviceset="WS2818" device=""/>
 <part name="GND3" library="supply1" deviceset="GND" device=""/>
-<part name="R4" library="rcl" deviceset="R-US_" device="R0201"/>
-<part name="R5" library="rcl" deviceset="R-US_" device="R0201"/>
-<part name="R6" library="rcl" deviceset="R-US_" device="R0201"/>
+<part name="R4" library="rcl" deviceset="R-US_" device="R0201" value="33Ω"/>
+<part name="R5" library="rcl" deviceset="R-US_" device="R0201" value="33Ω"/>
+<part name="R6" library="rcl" deviceset="R-US_" device="R0201" value="100Ω"/>
 <part name="P+4" library="supply1" deviceset="VCC" device=""/>
 <part name="U$3" library="Sparky" deviceset="4PAD" device=""/>
@@
 <instance part="C2" gate="G$1" x="2.54" y="116.84"/>
 <instance part="P+1" gate="VCC" x="25.4" y="121.92"/>
-<instance part="U$1" gate="G$1" x="25.4" y="106.68" rot="R270"/>
+<instance part="P1" gate="G$1" x="25.4" y="106.68" rot="R270"/>
 <instance part="P+3" gate="VCC" x="2.54" y="124.46"/>
 <instance part="GND1" gate="1" x="2.54" y="106.68"/>
-<instance part="U$2" gate="G$1" x="15.24" y="86.36"/>
+<instance part="U1" gate="G$1" x="15.24" y="86.36"/>
 <instance part="GND3" gate="1" x="30.48" y="81.28"/>
 <instance part="R4" gate="G$1" x="38.1" y="78.74"/>
@@
 <net name="VCC" class="0">
 <segment>
-<pinref part="U$1" gate="G$1" pin="1"/>
+<pinref part="P1" gate="G$1" pin="1"/>
 <pinref part="P+1" gate="VCC" pin="VCC"/>
 <wire x1="25.4" y1="114.3" x2="25.4" y2="119.38" width="0.1524" layer="91"/>
@@
 <net name="NEG_PAD" class="0">
 <segment>
-<pinref part="U$1" gate="G$1" pin="0"/>
+<pinref part="P1" gate="G$1" pin="0"/>
 <wire x1="27.94" y1="114.3" x2="27.94" y2="116.84" width="0.1524" layer="91"/>
 <label x="27.94" y="116.84" size="1.27" layer="95" rot="R90" xref="yes"/>
 </segment>
 <segment>
-<pinref part="U$2" gate="G$1" pin="OUTB"/>
+<pinref part="U1" gate="G$1" pin="OUTB"/>
 <wire x1="0" y1="83.82" x2="-5.08" y2="83.82" width="0.1524" layer="91"/>
-<pinref part="U$2" gate="G$1" pin="OUTG"/>
+<pinref part="U1" gate="G$1" pin="OUTG"/>
 <wire x1="0" y1="88.9" x2="-5.08" y2="88.9" width="0.1524" layer="91"/>
 <wire x1="-5.08" y1="83.82" x2="-5.08" y2="88.9" width="0.1524" layer="91"/>
-<pinref part="U$2" gate="G$1" pin="OUTR"/>
+<pinref part="U1" gate="G$1" pin="OUTR"/>
 <wire x1="0" y1="93.98" x2="-5.08" y2="93.98" width="0.1524" layer="91"/>
 <wire x1="-5.08" y1="88.9" x2="-5.08" y2="93.98" width="0.1524" layer="91"/>
@@
 </segment>
 <segment>
-<pinref part="U$2" gate="G$1" pin="GND"/>
+<pinref part="U1" gate="G$1" pin="GND"/>
 <pinref part="GND3" gate="1" pin="GND"/>
 </segment>
@@
 <net name="N$4" class="0">
 <segment>
-<pinref part="U$2" gate="G$1" pin="DIN"/>
+<pinref part="U1" gate="G$1" pin="DIN"/>
 <pinref part="R4" gate="G$1" pin="1"/>
 <wire x1="33.02" y1="78.74" x2="30.48" y2="78.74" width="0.1524" layer="91"/>
@@
 <net name="N$5" class="0">
 <segment>
-<pinref part="U$2" gate="G$1" pin="DO"/>
+<pinref part="U1" gate="G$1" pin="DO"/>
 <pinref part="R5" gate="G$1" pin="2"/>
 </segment>
@@
 <net name="N$6" class="0">
 <segment>
-<pinref part="U$2" gate="G$1" pin="VDD"/>
+<pinref part="U1" gate="G$1" pin="VDD"/>
 <pinref part="R6" gate="G$1" pin="1"/>
 </segment>
@@
 <net name="BIN" class="0">
 <segment>
-<pinref part="U$2" gate="G$1" pin="BIN"/>
+<pinref part="U1" gate="G$1" pin="BIN"/>
 <wire x1="30.48" y1="88.9" x2="35.56" y2="88.9" width="0.1524" layer="91"/>
 <label x="35.56" y="88.9" size="1.27" layer="95" xref="yes"/>
